File: ice4pi.kicad_sch (KiCad schematic)
At the start: 43 parts, among them J2 Raspberry_Pi_2_3, J3 Conn_02x12_Top_Bottom, U6 SN75160BN, U7 SN75161BN

Commit message: Release etherenet4pizero-1.0
Parts:
- removed D7, D8: LED, LED_SMD:LED_0603_1608Metric, symbol Device:LED
- removed J3: Conn_02x12_Top_Bottom, ice4pi:centronix-24-male, symbol Connector_Generic:Conn_02x12_Top_Bottom
- removed R111, R112, R113, R114, R115, R116, R117, R118, R211, R212, R213, R214, R215, R216, R217, R218: 3.3K, Resistor_SMD:R_0402_1005Metric, symbol Device:R
- removed R121, R122, R123, R124, R125, R126, R127, R128, R221, R222, R223, R224, R225, R226, R227, R228: 6.2K, Resistor_SMD:R_0402_1005Metric, symbol Device:R
- removed U6: SN75160BN, Package_DIP:DIP-20_W7.62mm, symbol Interface:SN75160BN
- removed U7: SN75161BN, Package_DIP:DIP-20_W7.62mm, symbol ice4pi:SN75161BN
- added C1, C2, C8: 100 nF, Capacitor_SMD:C_0402_1005Metric, symbol Device:C
- added C3: 0.01uF, Capacitor_SMD:C_0402_1005Metric, symbol Device:C_Small
- added C4: 10uF, Capacitor_SMD:C_0402_1005Metric, symbol Device:C
- added J1: Conn_02x03, Connector_PinHeader_2.54mm:PinHeader_2x03_P2.54mm_Vertical, symbol Connector_Generic:Conn_02x03_Odd_Even
- added J3: USB_C_Receptacle_USB2.0, Connector_USB:USB_C_Receptacle_GCT_USB4105-xx-A_16P_TopMnt_Horizontal, symbol Connector:USB_C_Receptacle_USB2.0
- added J4: RJ45_Amphenol_RJMG1BD3B8K1ANR, Connector_RJ:RJ45_Amphenol_RJMG1BD3B8K1ANR, symbol Connector:RJ45_Amphenol_RJMG1BD3B8K1ANR
- added L1: L, Inductor_SMD:L_1210_3225Metric, symbol Device:L
- added R1, R2: 50, Resistor_SMD:R_0402_1005Metric, symbol Device:R
- added R10: 2.32K, Resistor_SMD:R_0402_1005Metric, symbol Device:R
- added R5: 0, Resistor_SMD:R_0402_1005Metric, symbol Device:R
- added R6, R7: 1K, Resistor_SMD:R_0402_1005Metric, symbol Device:R
- added R8: 10K, Capacitor_SMD:C_0402_1005Metric, symbol Device:R
- added R9: 5.1K, Resistor_SMD:R_0402_1005Metric, symbol Device:R
- added U1: ENC28J60x-SS, Package_SO:SSOP-28_5.3x10.2mm_P0.65mm, symbol Interface_Ethernet:ENC28J60x-SS
- added U2: DSC1001DE1-025.0000, Oscillator:Oscillator_SMD_Abracon_ASDMB-4Pin_2.5x2.0mm, symbol Oscillator:ASDMB-xxxMHz
- C5: renamed from C7; value 10 uF -> 100 nF
- C6: renamed from C33; value 220 nF -> 100 nF
- C7: renamed from C34; value 220 nF -> 100 nF
- R3, R4: value 1K -> 50; PN ERJ-2GEJ102X -> (none)
Connections:
- net +3.3V: now also C5.1, C6.1, C7.1, C3.1, C8.1, L1.1, R8.1, U1.15 (VDDTX), U1.19 (VDDRX), U1.20 (VDDPLL), U1.25 (VDDOSC), U1.28 (VDD), U2.1 (Standby), U2.4 (VDD)
- net +5V: now also J3.A4 (VBUS), J3.A9 (VBUS), J3.B4 (VBUS), J3.B9 (VBUS); no longer C5.1, C6.1, C7.1
- net GND: now also C1.2, C2.2, C3.2, C4.2, C8.2, J3.A1 (GND), J3.A12 (GND), J3.B1 (GND), J3.B12 (GND), J3.S1 (SHIELD), J4.13 (SHIELD), J4.L2 (LEDY_K), J4.L3 (LEDG_K), J4.R8 (GND), R10.2, R9.2, U1.11 (VSSRX), U1.18 (VSSTX), U1.2 (VSS), U1.21 (VSSPLL), U1.22 (VSSOSC), U2.2 (GND); no longer R3.2, R4.2
- net at R3.1: now also R4.1, C2.1, J4.R5 (RCT)
- net CTRL_LED: no longer names the net of J2.7 (GCLK0/GPIO4)
- net GPIB_ATN renamed INT0
- net INT0: now also J1.2 (Pin_2)
- net GPIB_DAV renamed SI
- net SI: now also U1.7 (SI)
- net GPIB_DC renamed CS0
- net CS0: now also J1.1 (Pin_1)
- net GPIB_DIO01: no longer names the net of J2.38 (GPIO20/MOSI1)
- net GPIB_DIO02 renamed INT1
- net INT1: now also J1.6 (Pin_6)
- net GPIB_DIO03: no longer names the net of J2.36 (GPIO16)
- net GPIB_DIO04: no longer names the net of J2.35 (GPIO19/MISO1)
- net GPIB_DIO05: no longer names the net of J2.33 (PWM1/GPIO13)
- net GPIB_DIO06: no longer names the net of J2.32 (PWM0/GPIO12)
- net GPIB_DIO07: no longer names the net of J2.31 (GCLK2/GPIO6)
- net GPIB_DIO08 renamed CLKOUT
- net CLKOUT: now also R5.1
- net GPIB_EOI renamed SO
- net SO: now also U1.6 (SO)
- net GPIB_IFC: no longer names the net of J2.15 (GPIO22)
- net GPIB_NDAC: no longer names the net of J2.16 (GPIO23)
- net GPIB_NRFD: no longer names the net of J2.18 (GPIO24)
- net GPIB_PE renamed CS1
- net CS1: now also J1.5 (Pin_5)
- net GPIB_REN: no longer names the net of J2.13 (GPIO27)
- net GPIB_SRQ renamed SCK
- net SCK: now also U1.8 (SCK)
- net GPIB_TE: no longer names the net of J2.12 (GPIO18/PWM0)
- new net: C1.1, J4.R4 (TCT), L1.2, R1.1, R2.1
- new net: J3.A5 (CC1), J3.B5 (CC2), R9.1
- new net: C4.1, U1.1 (VCAP)
- new net: R10.1, U1.14 (RBIAS)
- new net: U1.23 (OSC1), U2.3 (Out)
- new net: R5.2, U1.3 (CLKOUT)
- new net: J4.L1 (LEDY_A), R7.2
- new net: J4.L4 (LEDG_A), R6.2
- new net CS: J1.3 (Pin_3), R8.2, U1.9 (~{CS})
- new net INT: J1.4 (Pin_4), U1.4 (~{INT})
- new net LEDA: R6.1, U1.27 (LEDA)
- new net LEDB: R7.1, U1.26 (LEDB)
- new net TPIN+: J4.R3 (RD+), R3.2, U1.13 (TPIN+)
- new net TPIN-: J4.R6 (RD-), R4.2, U1.12 (TPIN-)
- new net TPOUT+: J4.R1 (TD+), R1.2, U1.17 (TPOUT+)
- new net TPOUT-: J4.R2 (TD-), R2.2, U1.16 (TPOUT-)
- no-connect marks 8 -> 22
Other:
- note added: "2 to 1 jumper array."
- note removed: "R111-R118 3.3K"
- note removed: "R121-R128 6.2K"
- note removed: "R211-R218 3K3"
- note removed: "R221-R228 6.2K"
- title: gpib4pi-2.1 -> ethernet4pizero-1.0
- moved on the sheet: C5, C6, C7

Commit message: Release ethernet4pizero-direct-spi-1.0
Parts:
- removed C3: 0.01uF, Capacitor_SMD:C_0402_1005Metric, symbol Device:C_Small
- removed C4: 10uF, Capacitor_SMD:C_0402_1005Metric, symbol Device:C
- removed C8: 100 nF, Capacitor_SMD:C_0402_1005Metric, symbol Device:C
- removed R5: 0, Resistor_SMD:R_0402_1005Metric, symbol Device:R
- removed R8: 10K, Capacitor_SMD:C_0402_1005Metric, symbol Device:R
- removed U1: ENC28J60x-SS, Package_SO:SSOP-28_5.3x10.2mm_P0.65mm, symbol Interface_Ethernet:ENC28J60x-SS
- removed U2: DSC1001DE1-025.0000, Oscillator:Oscillator_SMD_Abracon_ASDMB-4Pin_2.5x2.0mm, symbol Oscillator:ASDMB-xxxMHz
- added R11: 200, Resistor_SMD:R_0402_1005Metric, symbol Device:R
- added U1: SN74LV4T125, Package_SO:TSSOP-14_4.4x5mm_P0.65mm, symbol 74xx:SN74LV4T125
- added U2, U3: SN65HVD11HD, Package_SO:SOIC-8_3.9x4.9mm_P1.27mm, symbol Interface_UART:SN65HVD11HD
- R10: value 2.32K -> 200
Connections:
- net +3.3V: now also U1.14 (VCC), U2.8 (VCC), U3.2 (~{RE}), U3.3 (DE), U3.8 (VCC)
- net CS: now also U1.1, U1.4
- net GND: now also U1.7 (GND), U2.2 (~{RE}), U2.3 (DE), U2.5 (GND), U3.5 (GND); no longer R10.2
- net LEDA: now also J2.37 (GPIO26)
- net LEDB: now also J2.22 (GPIO25)
- net SI: now also U1.3
- net SO: now also U1.5
- net TPIN+: now also U2.6 (A)
- net TPIN-: now also U2.7 (B)
- net TPOUT+: now also R11.2
- net TPOUT-: now also R10.2
- net at R10.1: now also U3.7 (B)
- net INT: no longer names the net of J1.4 (Pin_4)
- net INT0: no longer names the net of J1.2 (Pin_2)
- net INT0: no longer J2.22 (GPIO25)
- net INT1: no longer names the net of J1.6 (Pin_6)
- net INT1: no longer J2.37 (GPIO26)
- new net: U1.6, U3.4 (D)
- new net: U1.2, U2.1 (R)
- new net: R11.1, U3.6 (A)
- no-connect marks 22 -> 25
Other:
- title: ethernet4pizero-1.0 -> ethernet4pizero-direct-spi-1.0
