File: ice4pi.kicad_sch (KiCad schematic)
At the start: 52 parts, among them J1 Pmod 2x6, J2 raspberry_pi_2_3_4_ordered, U1 ICE40HX1K-TQ144, U2 W25Q32JVSSIQ, U3 MIC5504-1.2YM5, U4 DSC1001DI1-012.0000

Commit message: Release ice4pi-gpib-2.4
Connections:
- net CTRL_LED: now reaches U1.37 (IOB_24)
- net GPIB_DIO01: now reaches U1.38 (IOB_25)
- net GPIB_DIO02: now reaches U1.39 (IOB_26)
- net GPIB_DIO03: now reaches U1.41 (IOB_27)
- net GPIB_DIO04: now reaches U1.42 (IOB_28)
- net GPIB_DIO05: now reaches U1.43 (IOB_29)
- net GPIB_DIO06: now reaches U1.44 (IOB_30)
- net GPIB_DIO07: now reaches U1.45 (IOB_31)
- net GPIB_DIO08: now reaches U1.47 (IOB_32)
- net GPIB_PE: now reaches U1.48 (IOB_33)
- net GPIB_TE: now reaches U1.49 (IOB_35_GBIN5)
- net GPIB_REN: now reaches U1.50 (IOB_36_GBIN4)
- net GPIB_IFC: now reaches U1.52 (IOB_34)
- net GPIB_NDAC: now reaches U1.56 (IOB_37)
- net GPIB_NRFD: now reaches U1.58 (IOB_38)
- net GPIB_DAV: now reaches U1.60 (IOB_39)
- net GPIB_EOI: now reaches U1.61 (IOB_40)
- net GPIB_ATN: now reaches U1.62 (IOB_41)
- net GPIB_SRQ: now reaches U1.63 (IOB_42_CBSEL0)
- net GPIB_DC: now reaches U1.64 (IOB_43_CBSEL1)
Other:
- added sheet gpib4ice (gpib4ice.kicad_sch)
