File: ice4pi.kicad_sch (KiCad schematic)
At the start: 56 parts, among them J1 Pmod 2x6, J2 raspberry_pi_2_3_4_ordered, U1 ICE40HX1K-TQ144, U2 W25Q32JVSSIQ, U3 LT3030, U4 DSC1001DI1-012.0000

Commit message: Release ice4pi-2.2
Parts:
- removed C5: 0.01uF, Capacitor_SMD:C_0402_1005Metric, symbol Device:C_Small
- removed R1: 1M, Resistor_SMD:R_0402_1005Metric, symbol Device:R
- removed R7: 100, Resistor_SMD:R_0402_1005Metric, symbol Device:R
- removed R9: 0.1, Resistor_SMD:R_0402_1005Metric, symbol Device:R
- removed U3: LT3030, ice4pi:TSSOP-20_4.4x6.5mm_P0.65mm, symbol ice4pi:LT3030
- added U3: MIC5504-1.2YM5, Package_TO_SOT_SMD:SOT-23-5, symbol Regulator_Linear:MIC5504-1.2YM5
Connections:
- net +1V2: now also C8.1, U3.5 (VOUT)
- net +5V: now also U3.1 (VIN)
- net GND: now also U3.2 (GND)
- no-connect marks 7 -> 0
Other:
- title: ice4pi-2.1 -> ice4pi-2.2
- moved on the sheet: C1

Commit message: Release ice4pi-2.3
Parts:
- J2: PN SSW-120-01-T-D-006 -> SSQ-120-03-T-D
Connections:
- net +5V: now also U3.3 (EN)
Other:
- title: ice4pi-2.2 -> ice4pi-2.3
Changed lines of the file:
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@@
   (paper "A4")
   (title_block
-    (title "ice4pi-2.2")
+    (title "ice4pi-2.3")
   )
   (junction (at 189.23 107.95) (diameter 0) (color 0 0 0 0)
@@
   (junction (at 36.83 21.59) (diameter 0) (color 0 0 0 0)
   )
+  (junction (at 45.72 129.54) (diameter 0) (color 0 0 0 0)
+  )
   (junction (at 214.63 38.1) (diameter 0) (color 0 0 0 0)
   )
@@
   )
   (wire (pts (xy 276.86 102.87) (xy 273.05 102.87))
+    (stroke (width 0) (type default) (color 0 0 0 0))
+  )
+  (wire (pts (xy 45.72 129.54) (xy 45.72 134.62))
     (stroke (width 0) (type default) (color 0 0 0 0))
   )
@@
       (effects (font (size 1.27 1.27)) hide)
     )
-    (property "PN" "SSW-120-01-T-D-006" (id 4) (at 168.91 132.08 0)
-      (effects (font (size 1.27 1.27)) hide)
-    )
+    (property "PN" "SSQ-120-03-T-D" (id 4) (at 168.91 132.08 0)
+      (effects (font (size 1.27 1.27)) hide)
+    )

Commit message: Release ice4pi-2.4
Other:
- title: ice4pi-2.3 -> ice4pi-2.4
Changed lines of the file:
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@@
   (paper "A4")
   (title_block
-    (title "ice4pi-2.3")
+    (title "ice4pi-2.4")
   )
   (junction (at 189.23 107.95) (diameter 0) (color 0 0 0 0)
