File: ice4pi.kicad_pcb (KiCad board)
At the start: 4 copper layers, 65 x 30 mm, 66 parts, among them J1 Pmod 2x6, J2 Raspberry_Pi_2_3, U1 ICE40HX1K-TQ144, U2 W25Q32JVSSIQ, U3 LT3030, U4 DSC1001DI1-012.0000, U5 TFDU4101-TR3

Commit message: Release ice4pi-spark-6x-sfp-1.2.1
Parts:
- removed C2, C32: 0.1uF, Capacitor_SMD:C_0402_1005Metric
- removed C31: 4.7uF, Capacitor_SMD:C_0402_1005Metric
- removed D1, D2, D3, D4, D5: LED, LED_SMD:LED_0402_1005Metric
- removed J1: Pmod 2x6, ice4pi:PinSocket_2x06_P2.54mm_Vertical_1to6_7to12
- removed R10, R11, R12, R13, R14: 1K, Resistor_SMD:R_0402_1005Metric
- removed R21, R22: 47, Resistor_SMD:R_0402_1005Metric
- removed U5: TFDU4101-TR3, ice4pi:TFDU4101-TR3
- added ?: , ice4pi:lightside-instruments-logo, F.Cu at (92.0, 98.5)
- added J3: Conn_02x30_Odd_Even, Connector_PinSocket_2.00mm:PinSocket_2x30_P2.00mm_Vertical, B.Cu at (52.5, 85.1)
- added M0: MountingHole_2.7mm_Pad, MountingHole:MountingHole_2.7mm_Pad, F.Cu at (53.5, 98.5)
- added M1: MountingHole_2.7mm_Pad, MountingHole:MountingHole_2.7mm_Pad, F.Cu at (130.5, 98.5)
- added M2: MountingHole_2.7mm_Pad, MountingHole:MountingHole_2.7mm_Pad, F.Cu at (130.5, 67.0)
- moved C14 1.97 mm to (69.0, 74.3)
- moved C21 0.13 mm to (71.1, 70.1)
Connections:
- U1 pad 101: Net-(U1-Pad101) -> P55
- U1 pad 102: Net-(U1-Pad102) -> P56
- U1 pad 104: Net-(U1-Pad104) -> P57
- U1 pad 105: IR_TXD -> P58
- U1 pad 106: IR_RXD -> P59
- U1 pad 107: IR_SD -> P60
- U1 pad 11: Net-(U1-Pad11) -> P1
- U1 pad 12: Net-(U1-Pad12) -> P2
- U1 pad 19: Net-(U1-Pad19) -> P3
- U1 pad 20: Net-(U1-Pad20) -> P4
- U1 pad 22: Net-(U1-Pad22) -> P5
- U1 pad 23: Net-(U1-Pad23) -> P6
- U1 pad 24: Net-(U1-Pad24) -> P7
- U1 pad 25: Net-(U1-Pad25) -> P8
- U1 pad 26: Net-(U1-Pad26) -> P9
- U1 pad 28: Net-(U1-Pad28) -> P10
- U1 pad 29: Net-(U1-Pad29) -> P11
- U1 pad 31: Net-(U1-Pad31) -> P12
- U1 pad 32: Net-(U1-Pad32) -> P13
- U1 pad 33: Net-(U1-Pad33) -> P14
- U1 pad 34: Net-(U1-Pad34) -> P15
- U1 pad 37: Net-(U1-Pad37) -> P16
- U1 pad 38: Net-(U1-Pad38) -> P17
- U1 pad 39: Net-(U1-Pad39) -> P18
- U1 pad 41: Net-(U1-Pad41) -> P19
- U1 pad 42: Net-(U1-Pad42) -> P20
- U1 pad 43: Net-(U1-Pad43) -> P21
- U1 pad 44: Net-(U1-Pad44) -> P22
- U1 pad 45: Net-(U1-Pad45) -> P23
- U1 pad 47: Net-(U1-Pad47) -> P24
- U1 pad 48: Net-(U1-Pad48) -> P25
- U1 pad 49: Net-(U1-Pad49) -> P26
- U1 pad 50: Net-(U1-Pad50) -> P27
- U1 pad 52: Net-(U1-Pad52) -> P28
- U1 pad 56: Net-(U1-Pad56) -> P29
- U1 pad 58: Net-(U1-Pad58) -> P30
- U1 pad 60: Net-(U1-Pad60) -> P31
- U1 pad 61: Net-(U1-Pad61) -> P32
- U1 pad 62: Net-(U1-Pad62) -> P33
- U1 pad 63: Net-(U1-Pad63) -> P34
- U1 pad 64: Net-(U1-Pad64) -> P35
- U1 pad 73: Net-(U1-Pad73) -> P36
- U1 pad 74: Net-(U1-Pad74) -> P37
- U1 pad 75: Net-(U1-Pad75) -> P38
- U1 pad 76: Net-(U1-Pad76) -> P39
- U1 pad 78: PIO1_02 -> P40
- U1 pad 79: PIO1_03 -> P41
- U1 pad 80: PIO1_04 -> P42
- U1 pad 81: PIO1_05 -> P43
- U1 pad 87: PIO1_06 -> P44
- U1 pad 88: PIO1_07 -> P45
- U1 pad 90: PIO1_08 -> P46
- U1 pad 91: PIO1_09 -> P47
- U1 pad 93: Net-(U1-Pad93) -> P48
- U1 pad 94: Net-(U1-Pad94) -> P49
- U1 pad 95: LED4 -> P50
- U1 pad 96: LED3 -> P51
- U1 pad 97: LED2 -> P52
- U1 pad 98: LED1 -> P53
- U1 pad 99: LED0 -> P54
Routing:
- net IR_SD: track 41.6 -> 0.00 mm, vias 2 -> 0
- net P1: track 0.00 -> 41.5 mm, vias 0 -> 1
- net P59: track 0.00 -> 35.1 mm
- net P60: track 0.00 -> 33.6 mm
- net P7: track 0.00 -> 33.5 mm, vias 0 -> 1
- net P57: track 0.00 -> 33.2 mm
- net P5: track 0.00 -> 32.7 mm, vias 0 -> 1
- net P58: track 0.00 -> 31.7 mm
- net P55: track 0.00 -> 30.8 mm
- net P6: track 0.00 -> 30.4 mm, vias 0 -> 1
- net IR_RXD: track 29.6 -> 0.00 mm
- net P56: track 0.00 -> 29.4 mm
- net P2: track 0.00 -> 29.0 mm, vias 0 -> 1
- net P53: track 0.00 -> 28.7 mm
- net IR_TXD: track 28.0 -> 0.00 mm
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Other:
- board size 65 x 30 mm -> 85 x 54 mm
- net class Thin added: clearance 0.2, trace_width 0.2, via_dia 0.6, via_drill 0.4
- board text added: "ice4pi ver. 1.2*"
- board text added: "ice4pi-spark-6x-sfp ver. 1.2.1 (ice4pi ver. 1.2 mod) - 60x 3.3V IOs on a 2mm header - Spark v.2 6x SFP+ low speed signal module compatible"
- board text removed: "ice4pi ver. 1.2"

Commit message: Release ice4ultra96-1.2-1
Parts:
- removed svg2mod: G***, ice4pi:lsi-logo-16mm
- added C2: 10uF, Capacitor_SMD:C_0402_1005Metric, F.Cu at (74.0, 87.0)
- added C7: 10uF, Capacitor_SMD:C_0402_1005Metric, F.Cu at (65.3, 91.7)
- added J1: Conn_02x20_Odd_Even, Connector_PinSocket_2.00mm:PinSocket_2x20_P2.00mm_Vertical, B.Cu at (124.5, 97.5)
- added M2: MountingHole_2.7mm_Pad, MountingHole:MountingHole_2.7mm_Pad, F.Cu at (53.5, 67.0)
- added R3: 0, Resistor_SMD:R_0402_1005Metric, F.Cu at (78.8, 94.6)
- added R4: 0, Resistor_SMD:R_0402_1005Metric, F.Cu at (78.8, 87.3)
- added U5: LD1117S33TR_SOT223, Package_TO_SOT_SMD:SOT-223-3_TabPin2, F.Cu at (70.8, 91.7)
- J3: value Conn_02x30_Odd_Even -> Conn_02x02_Odd_Even; footprint Connector_PinSocket_2.00mm:PinSocket_2x30_P2.00mm_Vertical -> Connector_PinHeader_2.54mm:PinHeader_2x02_P2.54mm_Vertical; moved to F.Cu
- moved R17 72.1 mm to (129.7, 80.3), turned to 180 degrees
- moved R2 70.7 mm to (129.7, 79.0), turned to 180 degrees
- moved U2 67.3 mm to (125.0, 79.7), turned to 0 degrees
- moved R16 65.4 mm to (120.7, 80.8), turned to 90 degrees
- moved C28 65.4 mm to (127.0, 76.4), turned to 180 degrees
- moved C4 65.3 mm to (117.8, 77.0), turned to 180 degrees
- moved R15 61.9 mm to (123.0, 76.4), turned to 180 degrees
- moved J3 28.2 mm to (79.8, 92.2), turned to 180 degrees
- moved ? 19.2 mm to (81.6, 82.4)
- moved C15 0.20 mm to (70.9, 60.6), turned to 0 degrees
Connections:
- C11 pad 1: +3V3 -> +1V8
- C12 pad 1: +3V3 -> +1V8
- C13 pad 1: +3V3 -> +1V8
- C18 pad 1: +3V3 -> +1V8
- C28 pad 1: +3V3 -> +1V8
- C4 pad 1: +3V3 -> +1V8
- C9 pad 1: +3V3 -> +1V8
- J2 pad 18: iCE_CREST -> old_creset
- J2 pad 19: iCE_MOSI -> old_mosi
- J2 pad 21: iCE_MISO -> old_miso
- J2 pad 22: iCE_CDONE -> old_cdone
- J2 pad 23: iCE_SCK -> old_sck
- J2 pad 24: iCE_SS_B -> old_ss_b
- J3 pad 1: P1 -> +3V3
- J3 pad 2: P2 -> +3.3VP
- J3 pad 3: P3 -> +5VP
- J3 pad 4: P4 -> +5V
- R15 pad 1: +3V3 -> +1V8
- R16 pad 1: +3V3 -> +1V8
- R17 pad 1: +3V3 -> +1V8
- R18 pad 1: +3V3 -> +1V8
- R19 pad 1: +3V3 -> +1V8
- R2 pad 1: +3V3 -> +1V8
- U1 pad 1: Net-(U1-Pad1) -> old_mosi
- U1 pad 10: Net-(U1-Pad10) -> old_ss_b
- U1 pad 100: +3V3 -> +1V8
- U1 pad 109: Net-(U1-Pad109) -> (no net)
- U1 pad 11: P1 -> (no net)
- U1 pad 110: Net-(U1-Pad110) -> (no net)
- U1 pad 12: P2 -> (no net)
- U1 pad 124: Net-(U1-Pad124) -> (no net)
- U1 pad 125: Net-(U1-Pad125) -> (no net)
- U1 pad 126: Net-(U1-Pad126) -> (no net)
- U1 pad 127: Net-(U1-Pad127) -> (no net)
- U1 pad 130: Net-(U1-Pad130) -> (no net)
- U1 pad 131: Net-(U1-Pad131) -> (no net)
- U1 pad 142: Net-(U1-Pad142) -> (no net)
- U1 pad 143: Net-(U1-Pad143) -> (no net)
- U1 pad 144: Net-(U1-Pad144) -> (no net)
- U1 pad 15: Net-(U1-Pad15) -> (no net)
- U1 pad 16: Net-(U1-Pad16) -> (no net)
- U1 pad 17: Net-(U1-Pad17) -> (no net)
- U1 pad 18: Net-(U1-Pad18) -> (no net)
- U1 pad 19: P3 -> (no net)
- U1 pad 2: Net-(U1-Pad2) -> old_creset
- U1 pad 20: P4 -> (no net)
- U1 pad 22: P5 -> (no net)
- U1 pad 23: P6 -> (no net)
- U1 pad 24: P7 -> (no net)
- U1 pad 25: P8 -> (no net)
- U1 pad 26: P9 -> (no net)
- U1 pad 28: P10 -> (no net)
- U1 pad 29: P11 -> (no net)
- U1 pad 3: Net-(U1-Pad3) -> old_cdone
- U1 pad 31: P12 -> (no net)
- U1 pad 32: P13 -> (no net)
- U1 pad 33: P14 -> (no net)
- U1 pad 34: P15 -> (no net)
- U1 pad 37: P16 -> (no net)
- U1 pad 38: P17 -> (no net)
- U1 pad 39: P18 -> (no net)
- U1 pad 4: Net-(U1-Pad4) -> old_miso
- U1 pad 40: Net-(U1-Pad40) -> (no net)
- U1 pad 41: P19 -> (no net)
- U1 pad 42: P20 -> (no net)
- U1 pad 43: P21 -> (no net)
- U1 pad 44: P22 -> (no net)
- U1 pad 45: P23 -> (no net)
- U1 pad 46: +3V3 -> +1V8
- U1 pad 47: P24 -> (no net)
- U1 pad 48: P25 -> (no net)
- U1 pad 49: P26 -> (no net)
- U1 pad 50: P27 -> (no net)
- U1 pad 52: P28 -> (no net)
- U1 pad 53: Net-(U1-Pad53) -> (no net)
- U1 pad 54: Net-(U1-Pad54) -> (no net)
- U1 pad 55: Net-(U1-Pad55) -> (no net)
- U1 pad 56: P29 -> (no net)
- U1 pad 57: +3V3 -> +1V8
- U1 pad 58: P30 -> (no net)
- U1 pad 60: P31 -> (no net)
- U1 pad 61: P32 -> (no net)
- U1 pad 62: P33 -> (no net)
- U1 pad 63: P34 -> (no net)
- U1 pad 7: Net-(U1-Pad7) -> old_sck
- U1 pad 72: +3V3 -> +1V8
- U1 pad 77: Net-(U1-Pad77) -> (no net)
- U1 pad 82: Net-(U1-Pad82) -> (no net)
- U1 pad 83: Net-(U1-Pad83) -> (no net)
- U1 pad 84: Net-(U1-Pad84) -> (no net)
- U1 pad 85: Net-(U1-Pad85) -> (no net)
- U1 pad 89: +3V3 -> +1V8
- U2 pad 8: +3V3 -> +1V8
- U3 pad 1: Net-(U3-Pad1) -> (no net)
- U3 pad 17: Net-(U3-Pad17) -> (no net)
- U3 pad 18: Net-(U3-Pad18) -> (no net)
- U3 pad 19: Net-(U3-Pad19) -> (no net)
- U3 pad 2: Net-(U3-Pad2) -> (no net)
- U3 pad 3: Net-(U3-Pad3) -> (no net)
- U3 pad 4: Net-(U3-Pad4) -> (no net)
Routing:
- net P1: track 41.5 -> 0.00 mm, vias 1 -> 0
- net old_mosi: track 0.00 -> 39.7 mm, vias 0 -> 1
- net +1V8: track 0.00 -> 38.5 mm, vias 0 -> 11
- net old_ss_b: track 0.00 -> 34.8 mm, vias 0 -> 1
- net +3V3: track 73.1 -> 39.4 mm, vias 21 -> 10
- net P7: track 33.5 -> 0.00 mm, vias 1 -> 0
- net P5: track 32.7 -> 0.00 mm, vias 1 -> 0
- net old_sck: track 0.00 -> 31.8 mm, vias 0 -> 1
- net P6: track 30.4 -> 0.00 mm, vias 1 -> 0
- net old_cdone: track 0.00 -> 29.8 mm, vias 0 -> 1
- net old_miso: track 0.00 -> 29.1 mm, vias 0 -> 1
- net P2: track 29.0 -> 0.00 mm, vias 1 -> 0
- net P3: track 27.8 -> 0.00 mm, vias 1 -> 0
- net P4: track 27.6 -> 0.00 mm, vias 1 -> 0
- net old_creset: track 0.00 -> 25.9 mm, vias 0 -> 1
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- added copper zone on In2.Cu, net +1V8
- added copper zone on In2.Cu, net +5V
Other:
- board text added: "P/N: ice4ultra96-1.2 REV: 1"
- board text removed: "ice4pi ver. 1.2*"
- board text removed: "ice4pi-spark-6x-sfp ver. 1.2.1 (ice4pi ver. 1.2 mod) - 60x 3.3V IOs on a 2mm header - Spark v.2 6x SFP+ low speed signal module compatible"

Commit message: Release ice4ultra96-1.2-2
Parts:
- added J4: Conn_02x20_Odd_Even, ice4pi:Pin_Header_SMD_2x20_Pitch2mm, B.Cu at (124.5, 97.5)
- J1: footprint Connector_PinSocket_2.00mm:PinSocket_2x20_P2.00mm_Vertical -> ice4pi:Socket_Strip_SMD_2x20_Pitch2mm; moved to F.Cu
- turned J1 to 270 degrees
Routing:
- net GND: track 129.5 -> 140.5 mm, vias 38 -> 42
- net +1V8: track 38.5 -> 46.8 mm, vias 11 -> 13
- net iCE_CDONE: track 44.0 -> 50.7 mm, vias 2 -> 3
- net +VDC: track 0.00 -> 6.20 mm, vias 0 -> 2
- net iCE_CREST: track 47.9 -> 54.0 mm, vias 2 -> 3
- net P37: track 26.8 -> 32.8 mm, vias 0 -> 1
- net P35: track 25.5 -> 31.5 mm, vias 0 -> 2
- net P42: track 32.5 -> 38.5 mm, vias 0 -> 1
- net P57: track 52.5 -> 58.5 mm, vias 0 -> 1
- net P51: track 44.5 -> 50.5 mm, vias 0 -> 1
- net P49: track 42.7 -> 48.7 mm, vias 0 -> 1
- net P47: track 40.3 -> 46.3 mm, vias 0 -> 1
- net P45: track 37.9 -> 43.9 mm, vias 0 -> 1
- net P39: track 28.7 -> 34.7 mm, vias 0 -> 1
- net +5VP: track 14.9 -> 19.3 mm, vias 0 -> 2
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
Commit message: Release gpsclock4ultra96-1.0-1
Parts:
- removed ?: , ice4pi:lightside-instruments-logo
- removed ? (x4): , ice4pi:mount_hole
- removed C10, C11, C13, C15, C27, C29, C6: 0.01uF, Capacitor_SMD:C_0402_1005Metric
- removed C12, C14, C18, C19, C21, C23, C24, C25, C26, C28, C9: 0.1uF, Capacitor_SMD:C_0402_1005Metric
- removed C16, C20, C30: 10uF, Capacitor_SMD:C_0402_1005Metric
- removed C17, C22: 1 uF, Capacitor_SMD:C_0402_1005Metric
- removed C8: 4.7uF, Capacitor_SMD:C_0402_1005Metric
- removed D6: CDBU0520, Diode_SMD:D_0603_1608Metric
- removed J3: Conn_02x02_Odd_Even, Connector_PinHeader_2.54mm:PinHeader_2x02_P2.54mm_Vertical
- removed R15, R16, R17, R18, R19: 10K, Resistor_SMD:R_0402_1005Metric
- removed R20: 100, Resistor_SMD:R_0402_1005Metric
- added BT1: Battery_Cell, ice4pi:BatteryHolder_Keystone_2450, F.Cu at (70.8, 76.7)
- added D1: D_TVS, Resistor_SMD:R_0402_1005Metric, F.Cu at (81.9, 58.4)
- added D2: D_TVS, Resistor_SMD:R_0402_1005Metric, F.Cu at (60.6, 58.5)
- added D3: LED, Diode_SMD:D_0603_1608Metric, F.Cu at (127.6, 74.1)
- added J5: Conn_01x01_Shielded, ice4pi:SMA_LINX_CONSMA002_Horizontal, F.Cu at (81.4, 53.6)
- added J6: Conn_01x01_Shielded, ice4pi:SMA_LINX_CONSMA002_Horizontal, F.Cu at (60.1, 53.6)
- added L1: 27nH, Inductor_SMD:L_0402_1005Metric, F.Cu at (119.0, 58.6)
- added Q1: Q_NPN_BEC_BRT, Package_TO_SOT_SMD:SOT-323_SC-70, F.Cu at (124.2, 74.1)
- added R10: 4K7, Resistor_SMD:R_0402_1005Metric, F.Cu at (132.2, 81.0)
- added R11: 4K7, Resistor_SMD:R_0402_1005Metric, F.Cu at (132.2, 82.3)
- added R5: 0R, Resistor_SMD:R_0402_1005Metric, F.Cu at (119.2, 86.9)
- added R6: 1K, Resistor_SMD:R_0603_1608Metric, F.Cu at (127.6, 72.5)
- added R8: 4K7, Resistor_SMD:R_0402_1005Metric, F.Cu at (124.5, 84.7)
- added U10: PCA9306, Package_SO:SO-8_3.9x4.9mm_P1.27mm, F.Cu at (127.2, 80.3)
- added U6: LEA-M8T, RF_GPS:ublox_LEA, F.Cu at (106.1, 70.7)
- added U7: SN74LV1T34DBVRG4, Package_TO_SOT_SMD:SOT-23-5, F.Cu at (110.0, 90.0)
- added U8: SN74LV1T34DBVRG4, Package_TO_SOT_SMD:SOT-23-5, F.Cu at (116.0, 90.0)
- added U9: SN74LV1T34DBVRG4, Package_TO_SOT_SMD:SOT-23-5, F.Cu at (122.0, 90.0)
- added svg2mod: G***, ice4pi:lsi-logo-16mm, F.Cu at (97.4, 53.6)
- C1: value 10uF -> 1uF; footprint Capacitor_SMD:C_0402_1005Metric -> Resistor_SMD:R_0402_1005Metric
- C3: value 0.1uF -> 1uF; moved to F.Cu
- C4: value 10uF -> 22pF; footprint Capacitor_SMD:C_0402_1005Metric -> Inductor_SMD:L_0402_1005Metric
- C5: value 0.01uF -> 1uF; footprint Capacitor_SMD:C_0402_1005Metric -> Resistor_SMD:R_0402_1005Metric
- J2: value Raspberry_Pi_2_3 -> Conn_01x01_Shielded; footprint ice4pi:PinSocket_2x20_P2.54mm_Vertical_1_04mm -> ice4pi:SMA_LINX_CONSMA002_Horizontal; moved to F.Cu
- R1: value 1M -> 51
- R2: value 10K -> 51
- R3: value 0 -> 10K
- R4: value 0 -> 10R; footprint Resistor_SMD:R_0402_1005Metric -> Resistor_SMD:R_1206_3216Metric
- R7: value 100 -> 4K7
- R9: value 0.1 -> 200K
- U1: value ICE40HX1K-TQ144 -> 74LVC1G125; footprint Package_QFP:TQFP-144_20x20mm_P0.5mm -> Package_SO:TSOP-5_1.65x3.05mm_P0.95mm
- U2: value W25Q32JVSSIQ -> 74LVC1G125; footprint Package_SO:SOIC-8_3.9x4.9mm_P1.27mm -> Package_SO:TSOP-5_1.65x3.05mm_P0.95mm
- U3: value LT3030 -> SN74LV1T34DBVRG4; footprint ice4pi:TSSOP-20_4.4x6.5mm_P0.65mm -> Package_TO_SOT_SMD:SOT-23-5
- U4: value DSC1001DI1-012.0000 -> SN74LV1T34DBVRG4; footprint Oscillator:Oscillator_SMD_Abracon_ASDMB-4Pin_2.5x2.0mm -> Package_TO_SOT_SMD:SOT-23-5
- moved R9 72.4 mm to (132.2, 79.7), turned to 0 degrees
- moved R2 71.6 mm to (60.6, 60.2), turned to 0 degrees
- moved R7 66.4 mm to (124.5, 83.6), turned to 0 degrees
- moved C1 56.0 mm to (103.7, 81.1), turned to 0 degrees
- moved J2 55.1 mm to (113.5, 53.6), turned to 0 degrees
- moved U3 51.2 mm to (98.0, 90.0), turned to 0 degrees
- moved C5 50.9 mm to (101.0, 90.0), turned to 0 degrees
- moved R4 47.1 mm to (119.5, 63.6), turned to 270 degrees
- moved U4 45.2 mm to (104.0, 90.0), turned to 0 degrees
- moved R3 42.4 mm to (120.5, 86.9), turned to 270 degrees
- moved C3 42.2 mm to (111.3, 81.5), turned to 270 degrees
- moved R1 29.8 mm to (81.8, 60.2), turned to 0 degrees
- moved U2 25.3 mm to (100.0, 84.0)
- moved U1 23.0 mm to (94.0, 84.0)
- moved C7 22.8 mm to (86.0, 82.0), turned to 90 degrees
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Connections:
- C1 pad 1: +5V -> +3V3
- C3 pad 1: +3V3 -> Net-(BT1-Pad1)
- C4 pad 1: +1V8 -> Net-(C4-Pad1)
- C4 pad 2: GND -> Net-(C4-Pad2)
- C5 pad 1: Net-(C5-Pad1) -> +1V8
- C5 pad 2: Net-(C5-Pad2) -> GND
- C7 pad 1: +3.3VP -> +3V3
- J1 pad 11: P54 -> HD_GPIO_4
- J1 pad 13: P53 -> HD_GPIO_5
- J1 pad 15: P52 -> LSEXP_I2C0_SCL
- J1 pad 17: P50 -> LSEXP_I2C0_SDA
- J1 pad 22: P45 -> HD_GPIO_12
- J1 pad 27: P41 -> MIO44_PS_GPIO1_4
- J1 pad 34: P35 -> HD_GPIO_15
- J1 pad 37: +5VP -> +5V
- J2 pad 1: +3V3 -> Net-(C4-Pad2)
- J2 pad 2: +5V -> GND
- J4 pad 11: P54 -> HD_GPIO_4
- J4 pad 13: P53 -> HD_GPIO_5
- J4 pad 15: P52 -> LSEXP_I2C0_SCL
- J4 pad 17: P50 -> LSEXP_I2C0_SDA
- J4 pad 22: P45 -> HD_GPIO_12
- J4 pad 27: P41 -> MIO44_PS_GPIO1_4
- J4 pad 34: P35 -> HD_GPIO_15
- J4 pad 37: +5VP -> +5V
- R1 pad 1: +5V -> Net-(D1-Pad1)
- R2 pad 1: +1V8 -> Net-(D2-Pad1)
- R3 pad 1: +3.3VP -> +3V3
- R3 pad 2: +3V3 -> Net-(R3-Pad2)
- R4 pad 1: +5V -> Net-(L1-Pad2)
- R4 pad 2: +5VP -> Net-(R4-Pad2)
- R7 pad 1: Net-(C5-Pad1) -> LSEXP_I2C0_SDA
- R7 pad 2: GND -> +1V8
- R9 pad 1: +1V2 -> Net-(R9-Pad1)
- R9 pad 2: Net-(C5-Pad1) -> +3V3
- U1 pad 1: old_mosi -> GND
- U1 pad 2: old_creset -> Net-(Q1-Pad1)
- U1 pad 3: old_cdone -> GND
- U1 pad 4: old_miso -> Net-(R1-Pad2)
- U1 pad 5: GND -> +3V3
- U2 pad 1: iCE_SS_B -> GND
- U2 pad 2: iCE_MISO -> Net-(U2-Pad2)
- U2 pad 3: Net-(R16-Pad2) -> GND
- U2 pad 4: GND -> Net-(R2-Pad2)
- U2 pad 5: iCE_MOSI -> +3V3
- U3 pad 2: (no net) -> Net-(Q1-Pad1)
- U3 pad 3: (no net) -> GND
- U3 pad 4: (no net) -> HD_GPIO_15
- U3 pad 5: GND -> +1V8
- U4 pad 1: +3V3 -> (no net)
- U4 pad 2: GND -> Net-(U4-Pad2)
- U4 pad 3: 12MHz -> GND
- U4 pad 4: +3V3 -> HD_GPIO_5
- U5 pad 2: +3.3VP -> +3V3
Routing:
- net GND: track 140.5 -> 28.1 mm, vias 42 -> 13
- net iCE_SCK: track 77.5 -> 4.35 mm, vias 3 -> 1
- net Net-(Q1-Pad1): track 0.00 -> 67.6 mm, vias 0 -> 4
- net iCE_MOSI: track 70.7 -> 4.35 mm, vias 3 -> 1
- net iCE_SS_B: track 65.4 -> 4.35 mm, vias 4 -> 1
- net iCE_MISO: track 63.9 -> 4.35 mm, vias 3 -> 1
- net Net-(R2-Pad2): track 1.75 -> 56.1 mm
- net P59: track 58.5 -> 5.48 mm
- net Net-(BT1-Pad1): track 0.00 -> 52.6 mm, vias 0 -> 2
- net P57: track 58.5 -> 6.00 mm
- net P60: track 56.4 -> 4.35 mm
- net P58: track 54.4 -> 4.35 mm
- net iCE_CREST: track 54.0 -> 4.35 mm, vias 3 -> 1
- net P54: track 49.1 -> 0.00 mm, vias 1 -> 0
- net +5V: track 57.4 -> 8.78 mm, vias 6 -> 1
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- added copper zone on B.Cu, net +1V8
- added copper zone on F.Cu, net GND
- removed copper zone on In2.Cu, net +1V2
- removed copper zone on In2.Cu, net +1V8
- removed copper zone on In2.Cu, net +5V
Other:
- outline, holes or cut-outs redrawn
- board text added: "1"
- board text added: "P/N:"
- board text added: "REV:"
- board text added: "gpsclock4ultra96-1"
- board text removed: "P/N: ice4ultra96-1.2 REV: 1"

Commit message: Release clockinput4ultra96-1.0-1
Parts:
- removed BT1: Battery_Cell, ice4pi:BatteryHolder_Keystone_2450
- removed C1: 1uF, Resistor_SMD:R_0402_1005Metric
- removed C2, C7: 10uF, Capacitor_SMD:C_0402_1005Metric
- removed C3: 1uF, Capacitor_SMD:C_0402_1005Metric
- removed C4: 22pF, Inductor_SMD:L_0402_1005Metric
- removed J2: Conn_01x01_Shielded, ice4pi:SMA_LINX_CONSMA002_Horizontal
- removed L1: 27nH, Inductor_SMD:L_0402_1005Metric
- removed R10, R11, R7, R8: 4K7, Resistor_SMD:R_0402_1005Metric
- removed R3: 10K, Resistor_SMD:R_0402_1005Metric
- removed R4: 10R, Resistor_SMD:R_1206_3216Metric
- removed R5: 0R, Resistor_SMD:R_0402_1005Metric
- removed R9: 200K, Resistor_SMD:R_0402_1005Metric
- removed U1, U2: 74LVC1G125, Package_SO:TSOP-5_1.65x3.05mm_P0.95mm
- removed U10: PCA9306, Package_SO:SO-8_3.9x4.9mm_P1.27mm
- removed U4, U7, U9: SN74LV1T34DBVRG4, Package_TO_SOT_SMD:SOT-23-5
- removed U5: LD1117S33TR_SOT223, Package_TO_SOT_SMD:SOT-223-3_TabPin2
- removed U6: LEA-M8T, RF_GPS:ublox_LEA
- removed the svg2mod at (97.4, 53.6)
- added C6: 1uF, Resistor_SMD:R_0402_1005Metric, F.Cu at (119.0, 90.0)
- added svg2mod: G***, ice4pi:lsi-logo-32mm, F.Cu at (106.8, 68.2)
Connections:
- Q1 pad 1: Net-(Q1-Pad1) -> Net-(D1-Pad1)
- R1 pad 2: Net-(R1-Pad2) -> GND
- R2 pad 2: Net-(R2-Pad2) -> GND
- R6 pad 1: +3V3 -> +5V
- U3 pad 2: Net-(Q1-Pad1) -> Net-(D1-Pad1)
- U8 pad 2: Net-(U2-Pad2) -> Net-(D2-Pad1)
Routing:
- net Net-(D1-Pad1): track 6.62 -> 81.0 mm, vias 0 -> 2
- net Net-(Q1-Pad1): track 67.6 -> 0.00 mm, vias 4 -> 0
- net Net-(D2-Pad1): track 6.60 -> 74.0 mm
- net Net-(R2-Pad2): track 56.1 -> 0.00 mm
- net Net-(BT1-Pad1): track 52.6 -> 0.00 mm, vias 2 -> 0
- net Net-(R1-Pad2): track 34.9 -> 0.00 mm
- net LSEXP_I2C0_SCL: track 38.2 -> 4.35 mm, vias 2 -> 1
- net +3V3: track 28.0 -> 0.00 mm, vias 12 -> 0
- net Net-(U2-Pad2): track 26.3 -> 0.00 mm
- net Net-(U6-Pad10): track 24.7 -> 0.00 mm, vias 2 -> 0
- net MIO44_PS_GPIO1_4: track 28.2 -> 4.35 mm, vias 3 -> 1
- net LSEXP_I2C0_SDA: track 26.7 -> 4.35 mm, vias 2 -> 1
- net Net-(U6-Pad4): track 17.7 -> 0.00 mm, vias 2 -> 0
- net Net-(U4-Pad2): track 15.7 -> 0.00 mm, vias 2 -> 0
- net GND: track 28.1 -> 15.9 mm, vias 13 -> 8
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- added copper zone on In2.Cu, net +5V
- removed copper zone on In2.Cu, net +3V3
Other:
- board text added: "1 PPS INPUT"
- board text added: "10 MHz -> pin 22, HDGC_GPIO_12 (D5) 1 PPS -> pin 34, HDGC_GPIO_15 (C5)"
- board text added: "10 MHz INPUT"
- board text added: "3.3V TTL 50 Ohm"
- board text added: ":"
- board text added: "P/N"
- board text added: "REV"
- board text added: "clockinput4ultra96-1"
- board text removed: "P/N:"
- board text removed: "REV:"
- board text removed: "gpsclock4ultra96-1"

Commit message: Release clockinput4ultra96-1.1
Other:
- net class Default removed
- net class Power removed
- net class Thin removed
- board text added: "clockinput4ultra96-1.1"
- board text removed: "1"
- board text removed: ":"
- board text removed: "P/N"
- board text removed: "REV"
- board text removed: "clockinput4ultra96-1"
