File: ice4pi.kicad_pcb (KiCad board)
At the start: 4 copper layers, 85 x 54 mm, 43 parts, among them J1 Conn_02x20_Odd_Even, J2 Conn_01x01_Shielded, J4 Conn_02x20_Odd_Even, J5 Conn_01x01_Shielded, J6 Conn_01x01_Shielded, M0 MountingHole_2.7mm_Pad, M1 MountingHole_2.7mm_Pad, M2 MountingHole_2.7mm_Pad, Q1 Q_NPN_BEC_BRT, U1 74LVC1G125, U10 PCA9306, U2 74LVC1G125, U3 SN74LV1T34DBVRG4, U4 SN74LV1T34DBVRG4, U5 LD1117S33TR_SOT223, U6 LEA-M8T, U7 SN74LV1T34DBVRG4, U8 SN74LV1T34DBVRG4, U9 SN74LV1T34DBVRG4

Commit message: Release gpsclock4ultra96-1.1
Other:
- net class Default removed
- net class Power removed
- net class Thin removed
