File: ice4pi.kicad_pcb (KiCad board)
At the start: 4 copper layers, 65 x 30 mm, 66 parts, among them J1 Pmod 2x6, J2 Raspberry_Pi_2_3, U1 ICE40HX1K-TQ144, U2 W25Q32JVSSIQ, U3 LT3030, U4 DSC1001DI1-012.0000, U5 TFDU4101-TR3

Commit message: Release ice4pi-2.0
Parts:
- removed C31: 4.7uF, Capacitor_SMD:C_0402_1005Metric
- removed C32: 0.1uF, Capacitor_SMD:C_0402_1005Metric
- removed R21, R22: 47, Resistor_SMD:R_0402_1005Metric
- removed U5: TFDU4101-TR3, ice4pi:TFDU4101-TR3
- svg2mod: footprint ice4pi:lsi-logo-16mm -> ice4pi:lsi-logo-16mm-fcu
- moved C2 3.47 mm to (108.4, 59.0)
- moved J1 3.47 mm to (112.8, 70.3)
Connections:
- U1 pad 1: Net-(U1-Pad1) -> (no net)
- U1 pad 10: Net-(U1-Pad10) -> (no net)
- U1 pad 101: Net-(U1-Pad101) -> (no net)
- U1 pad 102: Net-(U1-Pad102) -> (no net)
- U1 pad 104: Net-(U1-Pad104) -> (no net)
- U1 pad 105: IR_TXD -> (no net)
- U1 pad 106: IR_RXD -> (no net)
- U1 pad 107: IR_SD -> (no net)
- U1 pad 109: Net-(U1-Pad109) -> (no net)
- U1 pad 11: Net-(U1-Pad11) -> (no net)
- U1 pad 110: Net-(U1-Pad110) -> (no net)
- U1 pad 12: Net-(U1-Pad12) -> (no net)
- U1 pad 124: Net-(U1-Pad124) -> (no net)
- U1 pad 125: Net-(U1-Pad125) -> (no net)
- U1 pad 126: Net-(U1-Pad126) -> (no net)
- U1 pad 127: Net-(U1-Pad127) -> (no net)
- U1 pad 130: Net-(U1-Pad130) -> (no net)
- U1 pad 131: Net-(U1-Pad131) -> (no net)
- U1 pad 142: Net-(U1-Pad142) -> (no net)
- U1 pad 143: Net-(U1-Pad143) -> (no net)
- U1 pad 144: Net-(U1-Pad144) -> (no net)
- U1 pad 15: Net-(U1-Pad15) -> (no net)
- U1 pad 16: Net-(U1-Pad16) -> (no net)
- U1 pad 17: Net-(U1-Pad17) -> (no net)
- U1 pad 18: Net-(U1-Pad18) -> (no net)
- U1 pad 19: Net-(U1-Pad19) -> (no net)
- U1 pad 2: Net-(U1-Pad2) -> (no net)
- U1 pad 20: Net-(U1-Pad20) -> (no net)
- U1 pad 22: Net-(U1-Pad22) -> (no net)
- U1 pad 23: Net-(U1-Pad23) -> (no net)
- U1 pad 24: Net-(U1-Pad24) -> (no net)
- U1 pad 25: Net-(U1-Pad25) -> (no net)
- U1 pad 26: Net-(U1-Pad26) -> (no net)
- U1 pad 28: Net-(U1-Pad28) -> (no net)
- U1 pad 29: Net-(U1-Pad29) -> (no net)
- U1 pad 3: Net-(U1-Pad3) -> (no net)
- U1 pad 31: Net-(U1-Pad31) -> (no net)
- U1 pad 32: Net-(U1-Pad32) -> (no net)
- U1 pad 33: Net-(U1-Pad33) -> (no net)
- U1 pad 34: Net-(U1-Pad34) -> (no net)
- U1 pad 37: Net-(U1-Pad37) -> (no net)
- U1 pad 38: Net-(U1-Pad38) -> (no net)
- U1 pad 39: Net-(U1-Pad39) -> (no net)
- U1 pad 4: Net-(U1-Pad4) -> (no net)
- U1 pad 40: Net-(U1-Pad40) -> (no net)
- U1 pad 41: Net-(U1-Pad41) -> (no net)
- U1 pad 42: Net-(U1-Pad42) -> (no net)
- U1 pad 43: Net-(U1-Pad43) -> (no net)
- U1 pad 44: Net-(U1-Pad44) -> (no net)
- U1 pad 45: Net-(U1-Pad45) -> (no net)
- U1 pad 47: Net-(U1-Pad47) -> (no net)
- U1 pad 48: Net-(U1-Pad48) -> (no net)
- U1 pad 49: Net-(U1-Pad49) -> (no net)
- U1 pad 50: Net-(U1-Pad50) -> (no net)
- U1 pad 52: Net-(U1-Pad52) -> (no net)
- U1 pad 53: Net-(U1-Pad53) -> (no net)
- U1 pad 54: Net-(U1-Pad54) -> (no net)
- U1 pad 55: Net-(U1-Pad55) -> (no net)
- U1 pad 56: Net-(U1-Pad56) -> (no net)
- U1 pad 58: Net-(U1-Pad58) -> (no net)
- U1 pad 60: Net-(U1-Pad60) -> (no net)
- U1 pad 61: Net-(U1-Pad61) -> (no net)
- U1 pad 62: Net-(U1-Pad62) -> (no net)
- U1 pad 63: Net-(U1-Pad63) -> (no net)
- U1 pad 64: Net-(U1-Pad64) -> (no net)
- U1 pad 7: Net-(U1-Pad7) -> (no net)
- U1 pad 73: Net-(U1-Pad73) -> (no net)
- U1 pad 74: Net-(U1-Pad74) -> (no net)
- U1 pad 75: Net-(U1-Pad75) -> (no net)
- U1 pad 76: Net-(U1-Pad76) -> (no net)
- U1 pad 77: Net-(U1-Pad77) -> (no net)
- U1 pad 82: Net-(U1-Pad82) -> (no net)
- U1 pad 83: Net-(U1-Pad83) -> (no net)
- U1 pad 84: Net-(U1-Pad84) -> (no net)
- U1 pad 85: Net-(U1-Pad85) -> (no net)
- U1 pad 93: Net-(U1-Pad93) -> (no net)
- U1 pad 94: Net-(U1-Pad94) -> (no net)
- U3 pad 1: Net-(U3-Pad1) -> (no net)
- U3 pad 17: Net-(U3-Pad17) -> (no net)
- U3 pad 18: Net-(U3-Pad18) -> (no net)
- U3 pad 19: Net-(U3-Pad19) -> (no net)
- U3 pad 2: Net-(U3-Pad2) -> (no net)
- U3 pad 3: Net-(U3-Pad3) -> (no net)
- U3 pad 4: Net-(U3-Pad4) -> (no net)
Routing:
- net GND: track 134.7 -> 56.8 mm
- net +5V: track 46.9 -> 4.36 mm
- net IR_SD: track 41.6 -> 0.00 mm, vias 2 -> 0
- net IR_RXD: track 29.6 -> 0.00 mm
- net IR_TXD: track 28.0 -> 0.00 mm
- net +1V2: track 46.8 -> 26.5 mm
- net +3V3: track 79.6 -> 60.9 mm, vias 23 -> 21
- net Net-(C32-Pad1): track 9.04 -> 0.00 mm, vias 1 -> 0
- net Net-(C31-Pad2): track 4.99 -> 0.00 mm, vias 1 -> 0
- net PIO1_02: track 22.4 -> 26.0 mm, vias 0 -> 1
- net PIO1_04: track 25.1 -> 28.5 mm
- net PIO1_09: track 25.2 -> 28.7 mm
- net PIO1_08: track 23.3 -> 26.8 mm
- net PIO1_07: track 21.1 -> 24.6 mm
- net PIO1_05: track 27.7 -> 31.1 mm
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- added copper zone on F.Cu, net +1V2
- added copper zone on F.Cu, net +3V3
- added copper zone on B.Cu, net +5V
- added copper zone on F.Cu, net +5V
- added copper zone on F.Cu, net GND
Other:
- board text added: "3.3V"
- board text added: "GND"
- board text added: "IO1"
- board text added: "IO2"
- board text added: "IO3"
- board text added: "IO4"
- board text added: "IO5"
- board text added: "IO6"
- board text added: "IO7"
- board text added: "IO8"
- board text added: "PMOD"
- board text added: "ice4pi ver. 2.0"
- board text removed: "ice4pi ver. 1.2"

Commit message: Release ice4pi-2.1
Parts:
- J2: value Raspberry_Pi_2_3 -> raspberry_pi_2_3_4_ordered
Connections:
- U1 pad 1: (no net) -> unconnected-(U1-Pad1)
- U1 pad 10: (no net) -> unconnected-(U1-Pad10)
- U1 pad 101: (no net) -> unconnected-(U1-Pad101)
- U1 pad 102: (no net) -> unconnected-(U1-Pad102)
- U1 pad 104: (no net) -> unconnected-(U1-Pad104)
- U1 pad 105: (no net) -> IR_TXD
- U1 pad 106: (no net) -> IR_RXD
- U1 pad 107: (no net) -> IR_SD
- U1 pad 109: (no net) -> unconnected-(U1-Pad109)
- U1 pad 11: (no net) -> unconnected-(U1-Pad11)
- U1 pad 110: (no net) -> unconnected-(U1-Pad110)
- U1 pad 12: (no net) -> unconnected-(U1-Pad12)
- U1 pad 124: (no net) -> unconnected-(U1-Pad124)
- U1 pad 125: (no net) -> unconnected-(U1-Pad125)
- U1 pad 126: (no net) -> unconnected-(U1-Pad126)
- U1 pad 127: (no net) -> unconnected-(U1-Pad127)
- U1 pad 130: (no net) -> unconnected-(U1-Pad130)
- U1 pad 131: (no net) -> unconnected-(U1-Pad131)
- U1 pad 142: (no net) -> unconnected-(U1-Pad142)
- U1 pad 143: (no net) -> unconnected-(U1-Pad143)
- U1 pad 144: (no net) -> unconnected-(U1-Pad144)
- U1 pad 15: (no net) -> unconnected-(U1-Pad15)
- U1 pad 16: (no net) -> unconnected-(U1-Pad16)
- U1 pad 17: (no net) -> unconnected-(U1-Pad17)
- U1 pad 18: (no net) -> unconnected-(U1-Pad18)
- U1 pad 19: (no net) -> unconnected-(U1-Pad19)
- U1 pad 2: (no net) -> unconnected-(U1-Pad2)
- U1 pad 20: (no net) -> unconnected-(U1-Pad20)
- U1 pad 22: (no net) -> unconnected-(U1-Pad22)
- U1 pad 23: (no net) -> unconnected-(U1-Pad23)
- U1 pad 24: (no net) -> unconnected-(U1-Pad24)
- U1 pad 25: (no net) -> unconnected-(U1-Pad25)
- U1 pad 26: (no net) -> unconnected-(U1-Pad26)
- U1 pad 28: (no net) -> unconnected-(U1-Pad28)
- U1 pad 29: (no net) -> unconnected-(U1-Pad29)
- U1 pad 3: (no net) -> unconnected-(U1-Pad3)
- U1 pad 31: (no net) -> unconnected-(U1-Pad31)
- U1 pad 32: (no net) -> unconnected-(U1-Pad32)
- U1 pad 33: (no net) -> unconnected-(U1-Pad33)
- U1 pad 34: (no net) -> unconnected-(U1-Pad34)
- U1 pad 37: (no net) -> unconnected-(U1-Pad37)
- U1 pad 38: (no net) -> unconnected-(U1-Pad38)
- U1 pad 39: (no net) -> unconnected-(U1-Pad39)
- U1 pad 4: (no net) -> unconnected-(U1-Pad4)
- U1 pad 40: (no net) -> unconnected-(U1-Pad40)
- U1 pad 41: (no net) -> unconnected-(U1-Pad41)
- U1 pad 42: (no net) -> unconnected-(U1-Pad42)
- U1 pad 43: (no net) -> unconnected-(U1-Pad43)
- U1 pad 44: (no net) -> unconnected-(U1-Pad44)
- U1 pad 45: (no net) -> unconnected-(U1-Pad45)
- U1 pad 47: (no net) -> unconnected-(U1-Pad47)
- U1 pad 48: (no net) -> unconnected-(U1-Pad48)
- U1 pad 49: (no net) -> unconnected-(U1-Pad49)
- U1 pad 50: (no net) -> unconnected-(U1-Pad50)
- U1 pad 52: (no net) -> unconnected-(U1-Pad52)
- U1 pad 53: (no net) -> unconnected-(U1-Pad53)
- U1 pad 54: (no net) -> unconnected-(U1-Pad54)
- U1 pad 55: (no net) -> unconnected-(U1-Pad55)
- U1 pad 56: (no net) -> unconnected-(U1-Pad56)
- U1 pad 58: (no net) -> unconnected-(U1-Pad58)
- U1 pad 60: (no net) -> unconnected-(U1-Pad60)
- U1 pad 61: (no net) -> unconnected-(U1-Pad61)
- U1 pad 62: (no net) -> unconnected-(U1-Pad62)
- U1 pad 63: (no net) -> unconnected-(U1-Pad63)
- U1 pad 64: (no net) -> unconnected-(U1-Pad64)
- U1 pad 7: (no net) -> unconnected-(U1-Pad7)
- U1 pad 73: (no net) -> unconnected-(U1-Pad73)
- U1 pad 74: (no net) -> unconnected-(U1-Pad74)
- U1 pad 75: (no net) -> unconnected-(U1-Pad75)
- U1 pad 76: (no net) -> unconnected-(U1-Pad76)
- U1 pad 77: (no net) -> unconnected-(U1-Pad77)
- U1 pad 82: (no net) -> unconnected-(U1-Pad82)
- U1 pad 83: (no net) -> unconnected-(U1-Pad83)
- U1 pad 84: (no net) -> unconnected-(U1-Pad84)
- U1 pad 85: (no net) -> unconnected-(U1-Pad85)
- U1 pad 93: (no net) -> unconnected-(U1-Pad93)
- U1 pad 94: (no net) -> unconnected-(U1-Pad94)
- U3 pad 1: (no net) -> unconnected-(U3-Pad1)
- U3 pad 17: (no net) -> unconnected-(U3-Pad17)
- U3 pad 18: (no net) -> unconnected-(U3-Pad18)
- U3 pad 19: (no net) -> unconnected-(U3-Pad19)
- U3 pad 2: (no net) -> unconnected-(U3-Pad2)
- U3 pad 3: (no net) -> unconnected-(U3-Pad3)
- U3 pad 4: (no net) -> unconnected-(U3-Pad4)
Other:
- net class Default removed
- net class Power removed
- board text added: "ice4pi ver. 2.1"
- board text removed: "ice4pi ver. 2.0"

Commit message: Release ice4pi-2.2
Parts:
- removed C5: 0.01uF, Capacitor_SMD:C_0402_1005Metric
- removed R1: 1M, Resistor_SMD:R_0402_1005Metric
- removed R7: 100, Resistor_SMD:R_0402_1005Metric
- removed R9: 0.1, Resistor_SMD:R_0402_1005Metric
- U3: value LT3030 -> MIC5504-1.2YM5; footprint ice4pi:TSSOP-20_4.4x6.5mm_P0.65mm -> Package_TO_SOT_SMD:SOT-23-5
- turned U3 to 0 degrees
Connections:
- C8 pad 1: Net-(C5-Pad1) -> +1V2
- U3 pad 1: unconnected-(U3-Pad1) -> +5V
- U3 pad 2: unconnected-(U3-Pad2) -> GND
- U3 pad 5: GND -> +1V2
Routing:
- net Net-(C5-Pad1): track 10.7 -> 0.00 mm
- net +5V: track 4.36 -> 1.70 mm
- net Net-(C5-Pad2): track 1.75 -> 0.00 mm
- net Net-(R1-Pad2): track 1.65 -> 0.00 mm
- net GND: track 56.8 -> 55.7 mm
Other:
- board text added: "ice4pi ver. 2.2"
- board text removed: "ice4pi ver. 2.1"

Commit message: Release ice4pi-2.3
Parts:
- removed svg2mod: G***, ice4pi:lsi-logo-16mm-fcu
Connections:
- U3 pad 3: unconnected-(U3-Pad3) -> +5V
Routing:
- net +5V: track 1.70 -> 9.12 mm, vias 4 -> 5
Other:
- board text added: "ice4pi ver. 2.3"
- board text removed: "ice4pi ver. 2.2"

Commit message: Release ice4pi-2.4
Parts:
- added svg2mod: G***, ice4pi:lsi-logo-16mm-fcu, F.Cu at (99.3, 75.5)
Other:
- board text added: "ice4pi ver. 2.4"
- board text removed: "ice4pi ver. 2.3"
